File: nodemcu/nanoDRONE.sch (KiCad schematic (older format))
At the start: 10 parts, among them J1 3.7V, M1 Motor_DC, M2 Motor_DC, M3 Motor_DC, M4 Motor_DC, Q1 BC547, Q2 BC547, Q3 BC547, Q4 BC547, U1 NodeMCU_1.0_(ESP-12E)

Commit message: MPU6050 module integrated
Parts:
- added J2: MPU6050 Dev brd, Connector_Molex:Molex_KK-254_AE-6410-08A_1x08_P2.54mm_Vertical, symbol Connector_Generic:Conn_01x08
Connections:
- net at U1.24 (GND): now also J2.2 (Pin_2)
- net at U1.25 (3.3V): now also J2.1 (Pin_1)
- net at U1.28 (D2(GPIO4)): now also J2.4 (Pin_4)
- net at U1.29 (D1(GPIO5)): now also J2.3 (Pin_3)
Changed lines of the file:
@@
 Wire Wire Line
 	3150 4150 4350 4150
+$Comp
+L Connector_Generic:Conn_01x08 J2
+U 1 1 5FF16475
+P 6350 3550
+F 0 "J2" H 6430 3542 50  0000 L CNN
+F 1 "MPU6050 Dev brd" H 6430 3451 50  0000 L CNN
+F 2 "Connector_Molex:Molex_KK-254_AE-6410-08A_1x08_P2.54mm_Vertical" H 6350 3550 50  0001 C CNN
+F 3 "~" H 6350 3550 50  0001 C CNN
+	1    6350 3550
+	1    0    0    -1
+$EndComp
+Wire Wire Line
+	6150 3250 5950 3250
+Wire Wire Line
+	6150 3350 5950 3350
+Wire Wire Line
+	5950 2850 6100 2850
+Wire Wire Line
+	6100 2850 6100 3450
+Wire Wire Line
+	6100 3450 6150 3450
+Wire Wire Line
+	5950 2950 6050 2950
+Wire Wire Line
+	6050 2950 6050 3550
+Wire Wire Line
+	6050 3550 6150 3550
 $EndSCHEMATC
